File: eagle/env_follower.brd (EAGLE design)
At the start: 95 x 50 mm, 41 parts, among them IC1 TL084P, IC2 TL084P

Commit message: routed lfo
Parts:
- removed R17, R2: 100k, pot:3RP/1610N
- added LFO_LEVEL, LFO_RATE: 100k, pot:3RP/1610N
- C7: value (none) -> 1u
- moved R19 168.2 mm to (73.0, 19.0)
- moved LED2 167.8 mm to (66.0, 14.0), turned to 90 degrees
- moved LED1 160.0 mm to (60.0, 14.0), turned to 270 degrees
- moved S1 153.3 mm to (75.0, 8.00)
- moved R18 152.8 mm to (56.0, 20.0), turned to 90 degrees
- moved R16 148.1 mm to (69.0, 43.0), turned to 180 degrees
- moved R9 138.4 mm to (69.0, 46.0), turned to 180 degrees
- moved R15 137.9 mm to (58.0, 43.0), turned to 180 degrees
- moved R10 136.2 mm to (58.0, 46.0)
- moved R7 133.0 mm to (77.0, 42.0), turned to 90 degrees
- moved C7 121.6 mm to (82.0, 23.0), turned to 180 degrees
- moved R8 121.0 mm to (50.0, 43.0), turned to 270 degrees
- moved LFO_OUT 119.7 mm to (52.7, 0.20), turned to 180 degrees
- moved R6 117.0 mm to (86.0, 15.0), turned to 90 degrees
- moved R5 111.1 mm to (82.2, 14.9), turned to 270 degrees
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Connections:
- net GND: now also LFO_LEVEL.1; no longer R17.1
- net N$1: now also LFO_RATE.1; no longer R2.1
- net N$16: now also LFO_RATE.3; no longer R2.3
- net N$19: now also LFO_LEVEL.3; no longer R17.3
- net N$23: now also LFO_LEVEL.2; no longer R17.2
- net N$6: now also LFO_RATE.2; no longer R2.2
Routing:
- net GND: track 149.1 -> 277.4 mm
- net N$16: track 0.00 -> 80.9 mm
- net N$14: track 0.00 -> 70.2 mm
- net +12V: track 26.4 -> 82.1 mm, vias 0 -> 1
- net N$10: track 0.00 -> 42.7 mm, vias 0 -> 1
- net N$18: track 0.00 -> 39.1 mm, vias 0 -> 1
- net -12V: track 28.0 -> 66.6 mm
- net N$12: track 0.00 -> 36.5 mm
- net N$27: track 0.00 -> 31.6 mm
- net N$7: track 0.00 -> 27.5 mm
- net N$23: track 0.00 -> 25.2 mm
- net N$13: track 0.00 -> 15.1 mm
- net N$25: track 0.00 -> 14.6 mm
- net N$24: track 0.00 -> 10.1 mm
- net N$19: track 0.00 -> 9.66 mm
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
Commit message: layout tweaks
Parts:
- moved LFO_OUT 0.20 mm to (52.7, 0.00)
- renumbered R1 to TRACKING
Changed lines of the file:
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@@
 </element>
 <element name="PWR1" library="eurorack" package="POWER_16" value="POWER" x="18.05" y="45" smashed="yes" rot="R180">
-<attribute name="NAME" x="25.543" y="39.92" size="1.27" layer="25" ratio="10" rot="R180"/>
+<attribute name="NAME" x="7.543" y="39.92" size="1.27" layer="25" ratio="10" rot="R180"/>
 </element>
 <element name="U$2" library="adafruit" package="FB" value="FB" x="16.27" y="37.65" smashed="yes"/>
@@
 <attribute name="NAME" x="11.159" y="32.73" size="1.27" layer="25" ratio="10" rot="R180"/>
 <attribute name="POPULARITY" value="58" x="9" y="34" size="1.778" layer="27" rot="R180" display="off"/>
-<attribute name="VALUE" x="11.159" y="36.667" size="1.27" layer="27" ratio="10" rot="R180"/>
+<attribute name="VALUE" x="14.159" y="36.667" size="1.27" layer="27" ratio="10" rot="R180"/>
 </element>
 <element name="R11" library="rcl" package="0207/7" value="10k" x="8" y="26" smashed="yes" rot="R180">
@@
 <attribute name="VALUE" x="22.586" y="21.2588" size="1.27" layer="27" ratio="10" rot="R180"/>
 </element>
-<element name="R1" library="pot" library_urn="urn:adsk.eagle:library:331" package="3RP/1610N" package3d_urn="urn:adsk.eagle:package:22726/1" value="100k" x="33" y="4" smashed="yes">
-<attribute name="NAME" x="24.745" y="9.715" size="1.27" layer="25"/>
+<element name="TRACKING" library="pot" library_urn="urn:adsk.eagle:library:331" package="3RP/1610N" package3d_urn="urn:adsk.eagle:package:22726/1" value="100k" x="33" y="4" smashed="yes">
+<attribute name="NAME" x="25.545" y="7.415" size="1.27" layer="25"/>
 <attribute name="POPULARITY" value="8" x="33" y="4" size="1.778" layer="27" display="off"/>
-<attribute name="VALUE" x="29.825" y="6.54" size="1.27" layer="27"/>
+<attribute name="VALUE" x="36.725" y="5.84" size="1.27" layer="27"/>
 </element>
 <element name="AUDIO_IN" library="erthenvar" package="ERTHENVAR-JACK-90DEG" value="AUDIO-JACK" x="23" y="0" smashed="yes" rot="R180">
@@
 <attribute name="NAME" x="80.745" y="7.715" size="1.27" layer="25"/>
 <attribute name="POPULARITY" value="8" x="88" y="4" size="1.778" layer="27" display="off"/>
-<attribute name="VALUE" x="91.825" y="6.54" size="1.27" layer="27"/>
+<attribute name="VALUE" x="89.725" y="6.04" size="1.27" layer="27"/>
 </element>
 <element name="R5" library="rcl" package="0207/7" value="470" x="82.2" y="14.9" smashed="yes" rot="R270">
@@
 <attribute name="VALUE" x="65.825" y="6.54" size="1.27" layer="27"/>
 </element>
-<element name="LFO_OUT" library="erthenvar" package="ERTHENVAR-JACK-90DEG" value="AUDIO-JACK" x="52.7" y="0.2" smashed="yes" rot="R180">
-<attribute name="NAME" x="47.15" y="12.89" size="1.27" layer="21" rot="R270"/>
+<element name="LFO_OUT" library="erthenvar" package="ERTHENVAR-JACK-90DEG" value="AUDIO-JACK" x="52.7" y="0" smashed="yes" rot="R180">
+<attribute name="NAME" x="47.15" y="12.69" size="1.27" layer="21" rot="R270"/>
 </element>
 <element name="S1" library="switch" library_urn="urn:adsk.eagle:library:380" package="M9040P" package3d_urn="urn:adsk.eagle:package:27676/1" value="" x="75" y="8" smashed="yes">
@@
 <contactref element="R18" pad="1"/>
 <wire x1="42" y1="10" x2="42" y2="29.81" width="1.016" layer="1"/>
-<wire x1="47.7" y1="2.7" x2="42" y2="8.4" width="1.016" layer="1"/>
-<wire x1="42" y1="8.4" x2="42" y2="10" width="1.016" layer="1"/>
-<wire x1="47.7" y1="2.7" x2="49" y2="4" width="1.016" layer="1"/>
-<wire x1="49" y1="4" x2="57" y2="4" width="1.016" layer="1"/>
+<wire x1="47.7" y1="2.5" x2="42" y2="8.2" width="1.016" layer="1"/>
+<wire x1="42" y1="8.2" x2="42" y2="10" width="1.016" layer="1"/>
+<wire x1="47.7" y1="2.5" x2="49.2" y2="4" width="1.016" layer="1"/>
+<wire x1="49.2" y1="4" x2="57" y2="4" width="1.016" layer="1"/>
 <wire x1="57" y1="4" x2="56" y2="5" width="1.016" layer="1"/>
 <wire x1="56" y1="5" x2="56" y2="16.19" width="1.016" layer="1"/>
@@
 <contactref element="C3" pad="1"/>
 <contactref element="IC2" pad="12"/>
-<contactref element="R1" pad="2"/>
+<contactref element="TRACKING" pad="2"/>
 <wire x1="40" y1="24.19" x2="40" y2="19.81" width="1.016" layer="16"/>
 <wire x1="40" y1="19.81" x2="39.25" y2="19.06" width="1.016" layer="16"/>
@@
 <signal name="N$22">
 <contactref element="R14" pad="2"/>
-<contactref element="R1" pad="1"/>
+<contactref element="TRACKING" pad="1"/>
 <wire x1="28" y1="4" x2="28" y2="5" width="1.016" layer="16"/>
 <wire x1="28" y1="5" x2="25" y2="8" width="1.016" layer="16"/>
@@
 <contactref element="C7" pad="2"/>
 <contactref element="S1" pad="3"/>
-<wire x1="75" y1="3.301" x2="76.699" y2="5" width="1.016" layer="1"/>
-<wire x1="76.699" y1="5" x2="79" y2="5" width="1.016" layer="1"/>
-<wire x1="79" y1="5" x2="79.46" y2="5.46" width="1.016" layer="1"/>
+<wire x1="75" y1="3.301" x2="75.699" y2="4" width="1.016" layer="1"/>
+<wire x1="75.699" y1="4" x2="78" y2="4" width="1.016" layer="1"/>
+<wire x1="78" y1="4" x2="79.46" y2="5.46" width="1.016" layer="1"/>
 <wire x1="79.46" y1="5.46" x2="79.46" y2="23" width="1.016" layer="1"/>
 <wire x1="74.62" y1="35.81" x2="77" y2="38.19" width="1.016" layer="16"/>
@@
 <wire x1="47.7" y1="20.7" x2="47.7" y2="16.7004625" width="1.016" layer="1"/>
 <wire x1="47.7" y1="16.7004625" x2="47.6962" y2="16.6966625" width="1.016" layer="1"/>
-<wire x1="47.6962" y1="16.6966625" x2="47.7" y2="15.9" width="0" layer="19" extent="1-1"/>
+<wire x1="47.6962" y1="16.6966625" x2="47.7" y2="15.7" width="0" layer="19" extent="1-1"/>
 </signal>
 <signal name="N$19">
